File: hardware/interface/interface.sch (KiCad schematic (older format))
At the start: 7 parts, among them J1 Board Connector, SW1 Rotary_Encoder_Switch, U1 128x32_OLED, U2 MCP23018-E_SS

Commit message: Whoops; the connector should be on the back side of the board.
Connections:
- net +5V: now also J1.7 (Pin_7); no longer J1.1 (Pin_1)
- net GND: now also J1.1 (Pin_1); no longer J1.7 (Pin_7)
- net INT: now also J1.2 (Pin_2); no longer J1.8 (Pin_8)
- net SCL: now also J1.3 (Pin_3); no longer J1.5 (Pin_5)
- net SDA: now also J1.5 (Pin_5); no longer J1.3 (Pin_3)
Changed lines of the file:
@@
 $EndComp
 Wire Wire Line
-	2500 3550 1850 3550
+	2500 3550 2450 3550
 Wire Wire Line
 	1850 3550 1850 3500
 Wire Wire Line
-	2500 3850 1850 3850
+	2500 3850 2450 3850
 $Comp
 L power:GND #PWR0103
@@
 L Connector_Generic:Conn_02x04_Odd_Even J1
 U 1 1 602D01C9
-P 2700 3650
-F 0 "J1" H 2750 3967 50  0000 C CNN
-F 1 "Board Connector" H 2750 3876 50  0000 C CNN
-F 2 "Connector_IDC:IDC-Header_2x04_P2.54mm_Vertical" H 2700 3650 50  0001 C CNN
-F 3 "~" H 2700 3650 50  0001 C CNN
-	1    2700 3650
-	1    0    0    -1
-$EndComp
+P 2700 3750
+F 0 "J1" H 2750 4067 50  0000 C CNN
+F 1 "Board Connector" H 2750 3976 50  0000 C CNN
+F 2 "Connector_IDC:IDC-Header_2x04_P2.54mm_Vertical" H 2700 3750 50  0001 C CNN
+F 3 "~" H 2700 3750 50  0001 C CNN
+	1    2700 3750
+	1    0    0    1
+$EndComp
+Connection ~ 2400 3550
+Wire Wire Line
+	2400 3550 1850 3550
+Connection ~ 2450 3850
+Wire Wire Line
+	2450 3850 1850 3850
+Connection ~ 2450 3550
+Wire Wire Line
+	2450 3550 2400 3550
 $EndSCHEMATC
